Commit message: Offset controller eklnedi, robot front_wheel'e offset eklendi, teleop paketide eklendi, gazebo tarafında simülasyona belirli konumlara kutular eklendi.

File: src/tricycle_robot/gazebo_sim_model/gebot_urdf.xacro (robot description, xacro)
@@ -1,4 +1,7 @@
 <?xml version="1.0"?>
 <robot name="gebot" xmlns:xacro="http://www.ros.org/wiki/xacro">
+    <!-- Read controller lateral_offset directly from YAML so model and controller stay in sync -->
+    <xacro:property name="controller_config" value="${xacro.load_yaml('$(find tricycle_robot)/config/tricycle_controller.yaml')}"/>
+    <xacro:property name="lateral_offset" value="${controller_config['offset_tricycle_controller']['ros__parameters']['lateral_offset']}"/>
     <xacro:property name="base_width" value="0.9"/>
     <xacro:property name="base_length" value="1.35"/>
@@ -119,11 +122,4 @@
         <xacro:cylinder_inertia m="1" r="${wheel_radius}" h="${(wheel_width+0.02)}"/><!--5-->
     </link>
-    <!--<joint name="front_wheel_joint" type="continuous">
-        <axis xyz="0 0 1"/>
-        <parent link="base_chassis"/>
-        <child link="front_wheel"/>
-        <origin xyz="0.475 0.0 -0.145" rpy="${-pi/2} 0 0"/>
-        <dynamics damping="0.2" />
-    </joint>-->
     <!-- Steering Links and Joints-->
     <link name="steering_link">
@@ -143,11 +139,4 @@
         <xacro:cylinder_inertia m="1" r="0.02" h="0.93"/><!--0.01-->
     </link>
-    <!--<joint name="front_steering_joint" type="revolute">
-        <axis xyz="0 0 1"/>
-        <limit effort="1000.0" lower="-1.4" upper="1.4" velocity="0.5"/>
-        <parent link="base_chassis"/>
-        <child link="steering_link"/>
-        <origin xyz="0.65 0.0 0.4"/>
-    </joint>-->
     <joint name="front_steering_joint" type="fixed">
         <parent link="base_chassis"/>
@@ -155,25 +144,4 @@
         <origin xyz="0.65 0.0 0.4"/>
     </joint>
-    <!--<link name="chain_frame">
-        <visual>
-            <origin xyz="0.0 0.0 0.0" rpy="0.0 ${pi/2} 0.0"/>
-            <geometry>
-                <cylinder radius="0.01" length="0.2"/>
-            </geometry>
-            <material name="myblue"/>
-        </visual>
-        <collision>
-            <origin xyz="0.0 0.0 0.0" rpy="0.0 ${pi/2} 0.0"/>
-            <geometry>
-                <cylinder radius="0.01" length="0.2"/>
-            </geometry>
-        </collision>
-        <xacro:cylinder_inertia m="0.001" r="0.01" h="0.2"/>
-    </link>
-    <joint name="steering_gear"  type="fixed">
-        <parent link="steering_link"/>
-        <child link="chain_frame"/>
-        <origin xyz="-0.1 0.0 -0.465"/>
-    </joint>-->
     <link name="steering_wheel">
         <visual>
@@ -218,5 +186,6 @@
         <parent link="base_chassis"/>
         <child link="bearing"/>
-        <origin xyz="0.475 0.0 0.045"/><!--0.045-->
+        <!-- ROS frame: +Y is left. We map +lateral_offset to right by using negative Y. -->
+        <origin xyz="0.475 ${0.0 - lateral_offset} 0.045"/><!--0.045-->
     </joint>
     <link name="bearing_gear">
@@ -250,11 +219,4 @@
         <dynamics damping="0.2" />
     </joint>
-    <!--<joint name="front_wheel_joint" type="continuous">
-        <axis xyz="0 0 1" />
-        <parent link="chain_frame"/>
-        <child link="front_wheel"/>
-        <origin xyz="-0.1 0.0 -0.085" rpy="${-pi/2} ${pi/2} 0"/>
-        <dynamics damping="0.2" />
-    </joint>-->
     <!-- Gazebo Physics Parameters for Wheels -->
     <gazebo reference="front_wheel">

Commit message: IMU ve EKF eklendi.

File: src/tricycle_robot/gazebo_sim_model/gebot_urdf.xacro (robot description, xacro)
@@ -239,4 +239,37 @@
         <kd>1.0</kd>
     </gazebo>
+    <!-- IMU Sensor -->
+    <link name="imu_link">
+        <visual>
+            <geometry>
+                <box size="0.04 0.04 0.02"/>
+            </geometry>
+            <material name="black"/>
+        </visual>
+        <collision>
+            <geometry>
+                <box size="0.04 0.04 0.02"/>
+            </geometry>
+        </collision>
+        <xacro:box_inertia m="0.01" w="0.04" d="0.04" h="0.02"/>
+    </link>
+    <joint name="imu_joint" type="fixed">
+        <parent link="base_chassis"/>
+        <child link="imu_link"/>
+        <origin xyz="0.0 0.0 0.035" rpy="0 0 0"/>
+    </joint>
+    <gazebo reference="imu_link">
+        <sensor name="imu_sensor" type="imu">
+            <always_on>true</always_on>
+            <update_rate>50</update_rate>
+            <visualize>false</visualize>
+            <topic>/imu/data</topic>
+            <gz_frame_id>imu_link</gz_frame_id>
+        </sensor>
+    </gazebo>
+    <!-- Gazebo IMU system plugin (required for gz-sim) -->
+    <gazebo>
+        <plugin filename="gz-sim-imu-system" name="gz::sim::systems::Imu"/>
+    </gazebo>
     <!-- Include Gazebo Tricycle Control -->
     <xacro:include filename="$(find tricycle_robot)/gazebo_sim_model/gz_tricycle_control.xacro" />
