Commit message: base_link arka arksa getirildi

File: src/offset_tricycle_robot/urdf/forklift.urdf.xacro (robot description, xacro)
@@ -89,6 +89,7 @@
     <xacro:box_inertia m="10" w="${base_width}" d="${base_length}" h="${base_height}"/>
   </link>
+  <!-- base_link at rear axle center (odometry reference point); chassis origin is rear_axle_x ahead -->
   <joint name="base_link_joint" type="fixed">
-    <origin xyz="${-front_axle_x} 0.0 0.275" rpy="0.0 0.0 0.0"/>
+    <origin xyz="${-rear_axle_x} 0.0 0.275" rpy="0.0 0.0 0.0"/>
     <parent link="base_link"/>
     <child link="base_chassis"/>

Commit message: Robot renkleri düzenlendi.

File: src/offset_tricycle_robot/urdf/forklift.urdf.xacro (robot description, xacro)
@@ -51,22 +51,25 @@
     </inertial>
   </xacro:macro>
-  <!-- Materials (URDF visual) -->
+  <!-- Colors as properties: use in URDF materials and in Gazebo <ambient>/<diffuse> -->
+  <xacro:property name="color_black_rgba" value="0.0 0.0 0.0 1.0"/>
+  <xacro:property name="color_white_rgba" value="1.0 1.0 1.0 1.0"/>
+  <xacro:property name="color_blue_rgba" value="0.1 0.2 0.5 1.0"/>
+  <xacro:property name="color_gray_rgba" value="0.45 0.45 0.45 1.0"/>
+  <xacro:property name="color_red_rgba" value="0.8 0.0 0.0 1.0"/>
+  <!-- Materials (URDF / RViz): reference by material name in <visual> -->
   <material name="black">
-    <color rgba="0.0 0.0 0.0 1.0"/>
+    <color rgba="${color_black_rgba}"/>
   </material>
   <material name="white">
-    <color rgba="1.0 1.0 1.0 1.0"/>
+    <color rgba="${color_white_rgba}"/>
   </material>
-  <material name="wheel">
-    <color rgba="0.15 0.15 0.15 1.0"/>
+  <material name="blue">
+    <color rgba="${color_blue_rgba}"/>
   </material>
-  <material name="myblue">
-    <color rgba="0.0 0.0 0.5 1.0"/>
+  <material name="gray">
+    <color rgba="${color_gray_rgba}"/>
   </material>
-  <material name="base">
-    <color rgba="0.2 0.05 0.05 1.0"/>
-  </material>
-  <material name="lidar">
-    <color rgba="0.8 0.0 0.0 1.0"/>
+  <material name="red">
+    <color rgba="${color_red_rgba}"/>
   </material>
   <!-- Robot Base -->
@@ -85,5 +88,5 @@
         <box size="${base_length} ${base_width} ${base_height}"/>
       </geometry>
-      <material name="base"/>
+      <material name="gray"/>
     </visual>
     <xacro:box_inertia m="10" w="${base_width}" d="${base_length}" h="${base_height}"/>
@@ -101,5 +104,5 @@
         <box size="0.15 ${base_width} 0.3"/>
       </geometry>
-      <material name="lidar"/>
+      <material name="red"/>
     </visual>
     <collision>
@@ -127,5 +130,5 @@
           <cylinder radius="${rear_wheel_radius}" length="${rear_wheel_width}"/>
         </geometry>
-        <material name="wheel"/>
+        <material name="black"/>
       </visual>
       <xacro:cylinder_inertia m="1" r="${rear_wheel_radius}" h="${rear_wheel_width}"/>
@@ -147,5 +150,5 @@
         <cylinder radius="${front_right_drive_wheel_radius}" length="${front_right_drive_wheel_width}"/>
       </geometry>
-      <material name="wheel"/>
+      <material name="black"/>
     </visual>
     <collision>
@@ -162,5 +165,5 @@
         <cylinder radius="${front_left_wheel_radius}" length="${front_left_wheel_width}"/>
       </geometry>
-      <material name="wheel"/>
+      <material name="black"/>
     </visual>
     <collision>
@@ -185,5 +188,5 @@
         <cylinder radius="0.045" length="0.04"/>
       </geometry>
-      <material name="myblue"/>
+      <material name="blue"/>
     </visual>
     <collision>
@@ -209,5 +212,5 @@
         <cylinder radius="0.02" length="0.195"/>
       </geometry>
-      <material name="myblue"/>
+      <material name="blue"/>
     </visual>
     <collision>
@@ -220,5 +223,5 @@
   </link>
   <!-- Bearing_gear at chassis height (z=0 in base_chassis) -->
-  <joint name="drive_unit" type="fixed">
+  <joint name="bearing_gear_joint" type="fixed">
     <parent link="bearing"/>
     <child link="bearing_gear"/>
@@ -272,5 +275,5 @@
         <box size="0.04 0.04 0.02"/>
       </geometry>
-      <material name="black"/>
+      <material name="blue"/>
     </visual>
     <collision>
@@ -344,6 +347,14 @@
     <visual>
       <material>
-        <ambient>1.0 1.0 1.0 1</ambient>
-        <diffuse>1.0 1.0 1.0 1</diffuse>
+        <ambient>${color_gray_rgba}</ambient>
+        <diffuse>${color_gray_rgba}</diffuse>
+      </material>
+    </visual>
+  </gazebo>
+  <gazebo reference="front_panel">
+    <visual>
+      <material>
+        <ambient>${color_red_rgba}</ambient>
+        <diffuse>${color_red_rgba}</diffuse>
       </material>
     </visual>
@@ -352,6 +363,6 @@
     <visual>
       <material>
-        <ambient>0.3 0.3 0.3 1</ambient>
-        <diffuse>0.3 0.3 0.3 1</diffuse>
+        <ambient>${color_black_rgba}</ambient>
+        <diffuse>${color_black_rgba}</diffuse>
       </material>
     </visual>
@@ -360,6 +371,6 @@
     <visual>
       <material>
-        <ambient>0.3 0.3 0.3 1</ambient>
-        <diffuse>0.3 0.3 0.3 1</diffuse>
+        <ambient>${color_black_rgba}</ambient>
+        <diffuse>${color_black_rgba}</diffuse>
       </material>
     </visual>
@@ -368,6 +379,6 @@
     <visual>
       <material>
-        <ambient>0.3 0.3 0.3 1</ambient>
-        <diffuse>0.3 0.3 0.3 1</diffuse>
+        <ambient>${color_black_rgba}</ambient>
+        <diffuse>${color_black_rgba}</diffuse>
       </material>
     </visual>
@@ -376,6 +387,6 @@
     <visual>
       <material>
-        <ambient>0.3 0.3 0.3 1</ambient>
-        <diffuse>0.3 0.3 0.3 1</diffuse>
+        <ambient>${color_black_rgba}</ambient>
+        <diffuse>${color_black_rgba}</diffuse>
       </material>
     </visual>
@@ -384,6 +395,6 @@
     <visual>
       <material>
-        <ambient>0.1 0.1 0.1 1</ambient>
-        <diffuse>0.1 0.1 0.1 1</diffuse>
+        <ambient>${color_blue_rgba}</ambient>
+        <diffuse>${color_blue_rgba}</diffuse>
       </material>
     </visual>
@@ -392,30 +403,6 @@
     <visual>
       <material>
-        <ambient>0.9 0.9 0.0 1</ambient>
-        <diffuse>0.9 0.9 0.0 1</diffuse>
-      </material>
-    </visual>
-  </gazebo>
-  <gazebo reference="steering_link">
-    <visual>
-      <material>
-        <ambient>1.0 1.0 1.0 1</ambient>
-        <diffuse>1.0 1.0 1.0 1</diffuse>
-      </material>
-    </visual>
-  </gazebo>
-  <gazebo reference="steering_wheel">
-    <visual>
-      <material>
-        <ambient>0.1 0.1 0.1 1</ambient>
-        <diffuse>0.1 0.1 0.1 1</diffuse>
-      </material>
-    </visual>
-  </gazebo>
-  <gazebo reference="front_panel">
-    <visual>
-      <material>
-        <ambient>0.8 0.0 0.0 1</ambient>
-        <diffuse>0.8 0.0 0.0 1</diffuse>
+        <ambient>${color_blue_rgba}</ambient>
+        <diffuse>${color_blue_rgba}</diffuse>
       </material>
     </visual>

Commit message: Docker dosyaları eklendi.

File: src/offset_tricycle_robot/urdf/forklift.urdf.xacro (robot description, xacro)
@@ -275,5 +275,5 @@
         <box size="0.04 0.04 0.02"/>
       </geometry>
-      <material name="blue"/>
+      <material name="red"/>
     </visual>
     <collision>

Commit message: Lidar eklendi.

File: src/offset_tricycle_robot/urdf/forklift.urdf.xacro (robot description, xacro)
@@ -102,5 +102,5 @@
     <visual>
       <geometry>
-        <box size="0.15 ${base_width} 0.3"/>
+        <box size="0.20 ${base_width} 0.3"/>
       </geometry>
       <material name="red"/>
@@ -183,20 +183,6 @@
   <!-- Bearing (steering joint) – front right only -->
   <link name="bearing">
-    <visual>
-      <origin xyz="0.0 0.0 0.0" rpy="0.0 0.0 0.0"/>
-      <geometry>
-        <cylinder radius="0.045" length="0.04"/>
-      </geometry>
-      <material name="blue"/>
-    </visual>
-    <collision>
-      <origin xyz="0.0 0.0 0.0" rpy="0.0 0.0 0.0"/>
-      <geometry>
-        <cylinder radius="0.045" length="0.04"/>
-      </geometry>
-    </collision>
-    <xacro:cylinder_inertia m="1" r="0.0045" h="0.04"/>
-  </link>
-  <!-- Bearing at chassis top; z = base_height/2 so bearing_gear can sit at chassis center (z=0) -->
+    <xacro:cylinder_inertia m="0.1" r="0.045" h="0.04"/>
+  </link>
   <joint name="bearing_joint" type="revolute">
     <axis xyz="0 0 1"/>
@@ -206,32 +192,10 @@
     <origin xyz="${front_axle_x} ${-front_track_half} ${base_height/2}"/>
   </joint>
-  <link name="bearing_gear">
-    <visual>
-      <origin xyz="0.0 0.0 0.0" rpy="0.0 0.0 0.0"/>
-      <geometry>
-        <cylinder radius="0.02" length="0.195"/>
-      </geometry>
-      <material name="blue"/>
-    </visual>
-    <collision>
-      <origin xyz="0.0 0.0 0.0" rpy="0.0 0.0 0.0"/>
-      <geometry>
-        <cylinder radius="0.02" length="0.195"/>
-      </geometry>
-    </collision>
-    <xacro:cylinder_inertia m="1" r="0.02" h="0.195"/>
-  </link>
-  <!-- Bearing_gear at chassis height (z=0 in base_chassis) -->
-  <joint name="bearing_gear_joint" type="fixed">
-    <parent link="bearing"/>
-    <child link="bearing_gear"/>
-    <origin xyz="0.0 0.0 ${-base_height/2}"/>
-  </joint>
   <!-- Wheel center at same ground level as rear/front_left wheels -->
   <joint name="front_right_drive_wheel_joint" type="continuous">
     <axis xyz="0 0 1" />
-    <parent link="bearing_gear"/>
+    <parent link="bearing"/>
     <child link="front_right_drive_wheel"/>
-    <origin xyz="0.0 0.0 ${front_right_drive_wheel_center_z}" rpy="${-pi/2} 0.0 0.0"/>
+    <origin xyz="0.0 0.0 ${-base_height/2 + front_right_drive_wheel_center_z}" rpy="${-pi/2} 0.0 0.0"/>
     <dynamics damping="0.2" />
   </joint>
@@ -275,5 +239,5 @@
         <box size="0.04 0.04 0.02"/>
       </geometry>
-      <material name="red"/>
+      <material name="black"/>
     </visual>
     <collision>
@@ -301,4 +265,59 @@
   <gazebo>
     <plugin filename="gz-sim-imu-system" name="gz::sim::systems::Imu"/>
+  </gazebo>
+  <!-- LiDAR Sensor -->
+  <link name="lidar_link">
+    <visual>
+      <geometry>
+        <cylinder radius="0.05" length="0.04"/>
+      </geometry>
+      <material name="black"/>
+    </visual>
+    <collision>
+      <geometry>
+        <cylinder radius="0.05" length="0.04"/>
+      </geometry>
+    </collision>
+    <xacro:cylinder_inertia m="0.1" r="0.05" h="0.04"/>
+  </link>
+  <joint name="lidar_joint" type="fixed">
+    <parent link="front_panel"/>
+    <child link="lidar_link"/>
+    <origin xyz="0.0 0.0 ${0.15 + 0.02}" rpy="0 0 0"/>
+  </joint>
+  <gazebo reference="lidar_link">
+    <sensor name="gpu_lidar" type="gpu_lidar">
+      <always_on>true</always_on>
+      <update_rate>10</update_rate>
+      <visualize>true</visualize>
+      <topic>/scan</topic>
+      <gz_frame_id>lidar_link</gz_frame_id>
+      <ray>
+        <scan>
+          <horizontal>
+            <samples>720</samples>
+            <resolution>1</resolution>
+            <min_angle>-3.14159</min_angle>
+            <max_angle>3.14159</max_angle>
+          </horizontal>
+        </scan>
+        <range>
+          <min>0.1</min>
+          <max>12.0</max>
+          <resolution>0.01</resolution>
+        </range>
+        <noise>
+          <type>gaussian</type>
+          <mean>0.0</mean>
+          <stddev>0.01</stddev>
+        </noise>
+      </ray>
+    </sensor>
+  </gazebo>
+  <!-- Gazebo sensors system plugin (required for gpu_lidar) -->
+  <gazebo>
+    <plugin filename="gz-sim-sensors-system" name="gz::sim::systems::Sensors">
+      <render_engine>ogre2</render_engine>
+    </plugin>
   </gazebo>
   <!-- Gazebo ground truth odometry publisher -->
@@ -392,17 +411,9 @@
     </visual>
   </gazebo>
-  <gazebo reference="bearing">
-    <visual>
-      <material>
-        <ambient>${color_blue_rgba}</ambient>
-        <diffuse>${color_blue_rgba}</diffuse>
-      </material>
-    </visual>
-  </gazebo>
-  <gazebo reference="bearing_gear">
-    <visual>
-      <material>
-        <ambient>${color_blue_rgba}</ambient>
-        <diffuse>${color_blue_rgba}</diffuse>
+  <gazebo reference="lidar_link">
+    <visual>
+      <material>
+        <ambient>${color_black_rgba}</ambient>
+        <diffuse>${color_black_rgba}</diffuse>
       </material>
     </visual>
